File: sensors.kicad_sch (KiCad schematic)
At the start: 1 part, among them U1 GY-91 10 DOF Sensor

Commit message: Small ammendments
Parts:
- added C20: 10u, symbol Device:C
- added C21: 0.1u, symbol Device:C
- added R13, R14: 10k, symbol Device:R
Connections:
- net +3.3V_OUT: now reaches U1.2 (3.3V)
- net +3.3V_OUT: now also C20.1, C21.1, R13.1, R14.1
- net GND: now reaches U1.3 (GND)
- net GND: now also C20.2, C21.2
- net IMU_SCK: now reaches U1.4 (SCL/SCK)
- net IMU_MOSI: now reaches U1.5 (SDA/MOSI)
- net IMU_MISO: now reaches U1.6 (SAO/MISO)
- net IMU_CS: now reaches U1.7 (NCS)
- net IMU_CS: now also R14.2
- net BARO_CS: now reaches U1.8 (CSB)
- net BARO_CS: now also R13.2
- no-connect marks 0 -> 1

Commit message: 15.09.2026 - 21:22
Parts:
- C20, C21: footprint (none) -> Capacitor_SMD:C_0603_1608Metric_Pad1.08x0.95mm_HandSolder
- R13, R14: footprint (none) -> Resistor_SMD:R_0201_0603Metric_Pad0.64x0.40mm_HandSolder
Changed lines of the file:
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@@
 			)
 		)
-		(property "Footprint" ""
+		(property "Footprint" "Capacitor_SMD:C_0603_1608Metric_Pad1.08x0.95mm_HandSolder"
 			(at 41.6052 71.12 0)
 			(hide yes)
@@
 			)
 		)
-		(property "Footprint" ""
+		(property "Footprint" "Resistor_SMD:R_0201_0603Metric_Pad0.64x0.40mm_HandSolder"
 			(at 51.562 26.67 90)
 			(hide yes)
@@
 			)
 		)
-		(property "Footprint" ""
+		(property "Footprint" "Resistor_SMD:R_0201_0603Metric_Pad0.64x0.40mm_HandSolder"
 			(at 51.308 26.67 90)
 			(hide yes)
@@
 			)
 		)
-		(property "Footprint" ""
+		(property "Footprint" "Capacitor_SMD:C_0603_1608Metric_Pad1.08x0.95mm_HandSolder"
 			(at 33.3248 71.12 0)
 			(hide yes)

Commit message: 15.09.2026 21:50
Parts:
- R13, R14: footprint Resistor_SMD:R_0201_0603Metric_Pad0.64x0.40mm_HandSolder -> Resistor_SMD:R_0603_1608Metric_Pad0.98x0.95mm_HandSolder
Changed lines of the file:
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@@
 			)
 		)
-		(property "Footprint" "Resistor_SMD:R_0201_0603Metric_Pad0.64x0.40mm_HandSolder"
+		(property "Footprint" "Resistor_SMD:R_0603_1608Metric_Pad0.98x0.95mm_HandSolder"
 			(at 51.562 26.67 90)
 			(hide yes)
@@
 			)
 		)
-		(property "Footprint" "Resistor_SMD:R_0201_0603Metric_Pad0.64x0.40mm_HandSolder"
+		(property "Footprint" "Resistor_SMD:R_0603_1608Metric_Pad0.98x0.95mm_HandSolder"
 			(at 51.308 26.67 90)
 			(hide yes)
