File: ESP-FC Rev.0.0.kicad_pcb (KiCad board)
At the start: 2 copper layers, 45 parts, among them J1 USB_C_Receptacle, J2 BAT1_XT60, J3 Conn_01x02, J4 Conn_01x02, J5 Conn_01x02, J6 Conn_01x02, SW1 Push_Button, SW2 Push_Button, U1 GY-91 10 DOF Sensor, U2 ESP32-S3-WROOM-1, U3 INA180A2IDBVT, U4 TPS54336ADDA, U6 AMS1117-3.3

Commit message: 8.09.2026 - 20:26
Parts:
- added C23: 470u 50V, Capacitor_THT:CP_Radial_D10.0mm_P5.00mm, F.Cu at (200.4, 115.3)
- added C24: 470u 50V, Capacitor_THT:CP_Radial_D10.0mm_P5.00mm, F.Cu at (200.4, 126.8)
- added J10: M3, Connector_PinHeader_2.54mm:PinHeader_1x03_P2.54mm_Horizontal, F.Cu at (183.8, 140.8)
- added J7: M0, Connector_PinHeader_2.54mm:PinHeader_1x03_P2.54mm_Horizontal, F.Cu at (183.8, 111.8)
- added J8: M1, Connector_PinHeader_2.54mm:PinHeader_1x03_P2.54mm_Horizontal, F.Cu at (183.8, 121.5)
- added J9: M2, Connector_PinHeader_2.54mm:PinHeader_1x03_P2.54mm_Horizontal, F.Cu at (183.8, 131.1)
- C25, C26, C27, C28: value 4.7u -> 4.7u 50V; footprint Capacitor_SMD:C_0603_1608Metric -> Capacitor_SMD:C_1206_3216Metric_Pad1.33x1.80mm_HandSolder
- J2: footprint Connector_AMASS:AMASS_XT60-M_1x02_P7.20mm_Vertical -> Connector_AMASS:AMASS_XT60PW-M_1x02_P7.20mm_Horizontal
- moved J2 16.8 mm to (128.8, 130.0)
Connections:
- U2 pad 32: unconnected-(U2-MTCK/GPIO39/CLK_OUT3/SUBSPICS1-Pad32) -> M0
- U2 pad 33: unconnected-(U2-MTDO/GPIO40/CLK_OUT2-Pad33) -> M1
- U2 pad 34: unconnected-(U2-MTDI/GPIO41/CLK_OUT1-Pad34) -> M2
- U2 pad 35: unconnected-(U2-MTMS/GPIO42-Pad35) -> M3

Commit message: 8.09.2026 - 23:26
Changed lines of the file:
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@@
 		(embedded_fonts no)
+	)
+	(gr_line
+		(start 70 64)
+		(end 97 32)
+		(stroke
+			(width 0.2)
+			(type default)
+		)
+		(layer "F.Cu")
+	)
+	(gr_line
+		(start 70 132)
+		(end 70 64)
+		(stroke
+			(width 0.2)
+			(type default)
+		)
+		(layer "F.Cu")
+	)
+	(gr_line
+		(start 97 32)
+		(end 209 32)
+		(stroke
+			(width 0.2)
+			(type default)
+		)
+		(layer "F.Cu")
+	)
+	(gr_line
+		(start 104 163)
+		(end 70 132)
+		(stroke
+			(width 0.2)
+			(type default)
+		)
+		(layer "F.Cu")
+	)
+	(gr_line
+		(start 203 163)
+		(end 104 163)
+		(stroke
+			(width 0.2)
+			(type default)
+		)
+		(layer "F.Cu")
+	)
+	(gr_line
+		(start 209 32)
+		(end 252 70)
+		(stroke
+			(width 0.2)
+			(type default)
+		)
+		(layer "F.Cu")
+	)
+	(gr_line
+		(start 252 70)
+		(end 252 129)
+		(stroke
+			(width 0.2)
+			(type default)
+		)
+		(layer "F.Cu")
+	)
+	(gr_line
+		(start 252 129)
+		(end 203 163)
+		(stroke
+			(width 0.2)
+			(type default)
+		)
+		(layer "F.Cu")
 	)
 	(embedded_fonts no)

Commit message: 9.09.2026 - 00:29
Parts:
- added J11: Conn_01x10, Connector_JST:JST_GH_BM10B-GHS-TBT_1x10-1MP_P1.25mm_Vertical, F.Cu at (104.5, 139.3)
Connections:
- U2 pad 10: unconnected-(U2-GPIO17/U1TXD/ADC2_CH6-Pad10) -> GPS_RX
- U2 pad 11: unconnected-(U2-GPIO18/U1RXD/ADC2_CH7/CLK_OUT3-Pad11) -> GPS_TX
- U2 pad 12: unconnected-(U2-GPIO8/TOUCH8/ADC1_CH7/SUBSPICS1-Pad12) -> GPS_SDA
- U2 pad 17: unconnected-(U2-GPIO9/TOUCH9/ADC1_CH8/FSPIHD/SUBSPIHD-Pad17) -> GPS_SCL
- U2 pad 23: unconnected-(U2-GPIO21-Pad23) -> GPS_SFT_SWT
- U2 pad 24: unconnected-(U2-GPIO47/SPICLK_P/SUBSPICLK_P_DIFF-Pad24) -> Net-(U2-GPIO47/SPICLK_P/SUBSPICLK_P_DIFF)
- U2 pad 5: unconnected-(U2-GPIO5/TOUCH5/ADC1_CH4-Pad5) -> Net-(U2-GPIO5/TOUCH5/ADC1_CH4)
- U2 pad 9: unconnected-(U2-GPIO16/U0CTS/ADC2_CH5/XTAL_32K_N-Pad9) -> SBUS

Commit message: 15.09.2026 21:50
Parts:
- added C1: 1u, Capacitor_SMD:C_0603_1608Metric_Pad1.08x0.95mm_HandSolder, F.Cu at (41.8, 58.4)
- added C19: 4.7u, Capacitor_SMD:C_0805_2012Metric_Pad1.18x1.45mm_HandSolder, F.Cu at (54.1, 70.7)
- added C20: 10u, Capacitor_SMD:C_0603_1608Metric_Pad1.08x0.95mm_HandSolder, F.Cu at (53.9, 58.4)
- added C21: 0.1u, Capacitor_SMD:C_0603_1608Metric_Pad1.08x0.95mm_HandSolder, F.Cu at (53.9, 61.0)
- added C22: 100n, Capacitor_SMD:C_0603_1608Metric_Pad1.08x0.95mm_HandSolder, F.Cu at (60.3, 58.4)
- added C29: 100n, Capacitor_SMD:C_0603_1608Metric_Pad1.08x0.95mm_HandSolder, F.Cu at (41.8, 63.5)
- added C4: 0.1u, Capacitor_SMD:C_0603_1608Metric_Pad1.08x0.95mm_HandSolder, F.Cu at (41.8, 61.0)
- added J12: Conn_01x03, Connector_PinHeader_2.54mm:PinHeader_1x03_P2.54mm_Horizontal, F.Cu at (169.6, 150.0)
- added R10: 10k, Resistor_SMD:R_0603_1608Metric_Pad0.98x0.95mm_HandSolder, F.Cu at (41.8, 68.5)
- added R11: 5.1k, Resistor_SMD:R_0603_1608Metric_Pad0.98x0.95mm_HandSolder, F.Cu at (53.9, 73.5)
- added R12: 5.1k, Resistor_SMD:R_0603_1608Metric_Pad0.98x0.95mm_HandSolder, F.Cu at (53.9, 76.0)
- added R13: 10k, Resistor_SMD:R_0603_1608Metric_Pad0.98x0.95mm_HandSolder, F.Cu at (53.9, 63.5)
- added R14: 10k, Resistor_SMD:R_0603_1608Metric_Pad0.98x0.95mm_HandSolder, F.Cu at (53.9, 66.0)
- added R15: 100k, Resistor_SMD:R_0603_1608Metric_Pad0.98x0.95mm_HandSolder, F.Cu at (60.3, 61.0)
- added R16: 11k, Resistor_SMD:R_0603_1608Metric_Pad0.98x0.95mm_HandSolder, F.Cu at (60.3, 63.5)
- added R17: 110, Resistor_SMD:R_0603_1608Metric_Pad0.98x0.95mm_HandSolder, F.Cu at (41.8, 71.0)
- added R18: 10k, Resistor_SMD:R_0603_1608Metric_Pad0.98x0.95mm_HandSolder, F.Cu at (41.8, 73.5)
- added R19: 330, Resistor_SMD:R_0603_1608Metric_Pad0.98x0.95mm_HandSolder, F.Cu at (41.8, 76.0)
- added R5: 10k, Resistor_SMD:R_0603_1608Metric_Pad0.98x0.95mm_HandSolder, F.Cu at (41.8, 66.0)
- C10, C11, C13, C15, C17, C18, C3, C6, C9: footprint Capacitor_THT:C_Radial_D12.5mm_H25.0mm_P5.00mm -> Capacitor_SMD:C_0603_1608Metric_Pad1.08x0.95mm_HandSolder
- C12, C14, C16, C5, C7, C8: footprint Capacitor_THT:C_Radial_D12.5mm_H25.0mm_P5.00mm -> Capacitor_SMD:C_0805_2012Metric_Pad1.18x1.45mm_HandSolder
- C23, C24: footprint Capacitor_THT:CP_Radial_D10.0mm_P5.00mm -> Capacitor_SMD:C_1206_3216Metric_Pad1.33x1.80mm_HandSolder
- R3, R4, R6, R7, R8, R9: footprint RES_L500x_BRN:RES_L500x_BRN -> Resistor_SMD:R_0603_1608Metric_Pad0.98x0.95mm_HandSolder

Commit message: 15.09.2026 - 21:55
Parts:
- C23, C24: footprint Capacitor_SMD:C_1206_3216Metric_Pad1.33x1.80mm_HandSolder -> Capacitor_THT:CP_Radial_D10.0mm_P5.00mm
- U2: value ESP32-S3-WROOM-1 -> ESP32-S3-WROOM-1U

Commit message: 18.09.2026 20:58
Parts:
- removed the C23 at (132.2, 91.5)
- removed the C24 at (132.2, 103.0)
- C5: footprint Capacitor_SMD:C_0805_2012Metric_Pad1.18x1.45mm_HandSolder -> Capacitor_SMD:C_1206_3216Metric_Pad1.33x1.80mm_HandSolder
- C7, C8: footprint Capacitor_SMD:C_0805_2012Metric_Pad1.18x1.45mm_HandSolder -> Capacitor_SMD:C_1210_3225Metric_Pad1.33x2.70mm_HandSolder
- moved C24 4.19 mm to (200.0, 131.0)

Commit message: 19.09.2026 00:53
Parts:
- added J14: Conn_01x07, Connector_PinHeader_2.54mm:PinHeader_1x07_P2.54mm_Horizontal, F.Cu at (228.8, 124.8)
Connections:
- R19 pad 1: GPS_LED -> Net-(U2-GPIO47/SPICLK_P/SUBSPICLK_P_DIFF)
- R19 pad 2: Net-(U2-GPIO47/SPICLK_P/SUBSPICLK_P_DIFF) -> GPS_LED
- U2 pad 28: unconnected-(U2-SPIIO6/GPIO35/FSPID/SUBSPID-Pad28) -> LORA_M0
- U2 pad 29: unconnected-(U2-SPIIO7/GPIO36/FSPICLK/SUBSPICLK-Pad29) -> LORA_M1
- U2 pad 31: unconnected-(U2-GPIO38/FSPIWP/SUBSPIWP-Pad31) -> LORA_AUX
- U2 pad 36: unconnected-(U2-U0RXD/GPIO44/CLK_OUT2-Pad36) -> LORA_UART_TX
- U2 pad 37: unconnected-(U2-U0TXD/GPIO43/CLK_OUT1-Pad37) -> LORA_UART_RX
