File: mcu.kicad_sch (KiCad schematic)
At the start: 19 parts, among them J10 M3, J11 Conn_01x10, J12 Conn_01x03, J7 M0, J8 M1, J9 M2, SW1 Push_Button, SW2 Push_Button, U2 ESP32-S3-WROOM-1

Commit message: 15.09.2026 - 21:22
Parts:
- C1, C29, C4: footprint (none) -> Capacitor_SMD:C_0603_1608Metric_Pad1.08x0.95mm_HandSolder
- J12: footprint (none) -> Connector_PinHeader_1.00mm:PinHeader_1x03_P1.00mm_Horizontal
- R10, R17, R18, R19, R5: footprint (none) -> Resistor_SMD:R_0201_0603Metric_Pad0.64x0.40mm_HandSolder
Changed lines of the file:
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@@
 			)
 		)
-		(property "Footprint" ""
+		(property "Footprint" "Resistor_SMD:R_0201_0603Metric_Pad0.64x0.40mm_HandSolder"
 			(at 27.432 31.75 90)
 			(hide yes)
@@
 			)
 		)
-		(property "Footprint" ""
+		(property "Footprint" "Resistor_SMD:R_0201_0603Metric_Pad0.64x0.40mm_HandSolder"
 			(at 145.542 91.44 90)
 			(hide yes)
@@
 			)
 		)
-		(property "Footprint" ""
+		(property "Footprint" "Resistor_SMD:R_0201_0603Metric_Pad0.64x0.40mm_HandSolder"
 			(at 135.89 104.902 90)
 			(hide yes)
@@
 			)
 		)
-		(property "Footprint" ""
+		(property "Footprint" "Resistor_SMD:R_0201_0603Metric_Pad0.64x0.40mm_HandSolder"
 			(at 134.62 64.262 90)
 			(hide yes)
@@
 			)
 		)
-		(property "Footprint" ""
+		(property "Footprint" "Capacitor_SMD:C_0603_1608Metric_Pad1.08x0.95mm_HandSolder"
 			(at 153.9748 63.5 0)
 			(hide yes)
@@
 			)
 		)
-		(property "Footprint" ""
+		(property "Footprint" "Capacitor_SMD:C_0603_1608Metric_Pad1.08x0.95mm_HandSolder"
 			(at 146.3548 106.68 0)
 			(hide yes)
@@
 			)
 		)
-		(property "Footprint" ""
+		(property "Footprint" "Capacitor_SMD:C_0603_1608Metric_Pad1.08x0.95mm_HandSolder"
 			(at 30.1752 46.99 0)
 			(hide yes)
@@
 			)
 		)
-		(property "Footprint" ""
+		(property "Footprint" "Resistor_SMD:R_0201_0603Metric_Pad0.64x0.40mm_HandSolder"
 			(at 153.162 48.26 90)
 			(hide yes)
@@
 			)
 		)
-		(property "Footprint" ""
+		(property "Footprint" "Connector_PinHeader_1.00mm:PinHeader_1x03_P1.00mm_Horizontal"
 			(at 269.24 144.78 0)
 			(hide yes)

Commit message: 15.09.2026 21:50
Parts:
- C16: footprint Capacitor_THT:C_Radial_D12.5mm_H25.0mm_P5.00mm -> Capacitor_SMD:C_0805_2012Metric_Pad1.18x1.45mm_HandSolder
- C17: footprint Capacitor_THT:C_Radial_D12.5mm_H25.0mm_P5.00mm -> Capacitor_SMD:C_0603_1608Metric_Pad1.08x0.95mm_HandSolder
- J12: footprint Connector_PinHeader_1.00mm:PinHeader_1x03_P1.00mm_Horizontal -> Connector_PinHeader_2.54mm:PinHeader_1x03_P2.54mm_Horizontal
- R10, R17, R18, R19, R5: footprint Resistor_SMD:R_0201_0603Metric_Pad0.64x0.40mm_HandSolder -> Resistor_SMD:R_0603_1608Metric_Pad0.98x0.95mm_HandSolder
- U2: value ESP32-S3-WROOM-1 -> ESP32-S3-WROOM-1U
Connections:
- no-connect marks 4 -> 18
Changed lines of the file:
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@@
 	)
 	(no_connect
+		(at 129.54 38.1)
+	)
+	(no_connect
+		(at 129.54 60.96)
+	)
+	(no_connect
+		(at 129.54 40.64)
+	)
+	(no_connect
+		(at 129.54 104.14)
+	)
+	(no_connect
 		(at 262.89 29.21)
 	)
@@
 	)
 	(no_connect
+		(at 38.1 104.14)
+	)
+	(no_connect
+		(at 38.1 106.68)
+	)
+	(no_connect
+		(at 129.54 109.22)
+	)
+	(no_connect
+		(at 38.1 45.72)
+	)
+	(no_connect
+		(at 129.54 63.5)
+	)
+	(no_connect
+		(at 129.54 68.58)
+	)
+	(no_connect
+		(at 129.54 99.06)
+	)
+	(no_connect
 		(at 262.89 38.1)
 	)
@@
 		(at 262.89 55.88)
 	)
+	(no_connect
+		(at 38.1 109.22)
+	)
+	(no_connect
+		(at 129.54 101.6)
+	)
+	(no_connect
+		(at 129.54 71.12)
+	)
 	(wire
 		(pts
@@
 			)
 		)
-		(property "Footprint" "Resistor_SMD:R_0201_0603Metric_Pad0.64x0.40mm_HandSolder"
+		(property "Footprint" "Resistor_SMD:R_0603_1608Metric_Pad0.98x0.95mm_HandSolder"
 			(at 27.432 31.75 90)
 			(hide yes)
@@
 			)
 		)
-		(property "Footprint" "Resistor_SMD:R_0201_0603Metric_Pad0.64x0.40mm_HandSolder"
+		(property "Footprint" "Resistor_SMD:R_0603_1608Metric_Pad0.98x0.95mm_HandSolder"
 			(at 145.542 91.44 90)
 			(hide yes)
@@
 			)
 		)
-		(property "Value" "ESP32-S3-WROOM-1"
+		(property "Value" "ESP32-S3-WROOM-1U"
 			(at 85.9633 33.02 0)
 			(show_name no)
@@
 			)
 		)
-		(property "Footprint" "Capacitor_THT:C_Radial_D12.5mm_H25.0mm_P5.00mm"
+		(property "Footprint" "Capacitor_SMD:C_0603_1608Metric_Pad1.08x0.95mm_HandSolder"
 			(at 73.3552 26.67 0)
 			(hide yes)
@@
 			)
 		)
-		(property "Footprint" "Resistor_SMD:R_0201_0603Metric_Pad0.64x0.40mm_HandSolder"
+		(property "Footprint" "Resistor_SMD:R_0603_1608Metric_Pad0.98x0.95mm_HandSolder"
 			(at 135.89 104.902 90)
 			(hide yes)
@@
 			)
 		)
-		(property "Footprint" "Resistor_SMD:R_0201_0603Metric_Pad0.64x0.40mm_HandSolder"
+		(property "Footprint" "Resistor_SMD:R_0603_1608Metric_Pad0.98x0.95mm_HandSolder"
 			(at 134.62 64.262 90)
 			(hide yes)
@@
 			)
 		)
-		(property "Footprint" "Capacitor_THT:C_Radial_D12.5mm_H25.0mm_P5.00mm"
+		(property "Footprint" "Capacitor_SMD:C_0805_2012Metric_Pad1.18x1.45mm_HandSolder"
 			(at 65.7352 26.67 0)
 			(hide yes)
@@
 			)
 		)
-		(property "Footprint" "Resistor_SMD:R_0201_0603Metric_Pad0.64x0.40mm_HandSolder"
+		(property "Footprint" "Resistor_SMD:R_0603_1608Metric_Pad0.98x0.95mm_HandSolder"
 			(at 153.162 48.26 90)
 			(hide yes)
@@
 			)
 		)
-		(property "Footprint" "Connector_PinHeader_1.00mm:PinHeader_1x03_P1.00mm_Horizontal"
+		(property "Footprint" "Connector_PinHeader_2.54mm:PinHeader_1x03_P2.54mm_Horizontal"
 			(at 269.24 144.78 0)
 			(hide yes)

Commit message: 19.09.2026 00:53
Parts:
- added J14: Conn_01x07, Connector_PinHeader_2.54mm:PinHeader_1x07_P2.54mm_Horizontal, symbol Connector_Generic:Conn_01x07
Connections:
- net +3.3V_OUT: now also J14.6 (Pin_6)
- net GND: now also J14.7 (Pin_7)
- net GPS_LED: now also R19.2; no longer R19.1
- net at U2.24 (GPIO47/SPICLK_P/SUBSPICLK_P_DIFF): now also R19.1; no longer R19.2
- net LORA_M0: now reaches U2.28 (SPIIO6/GPIO35/FSPID/SUBSPID)
- net LORA_M0: now also J14.1 (Pin_1)
- net LORA_M1: now reaches U2.29 (SPIIO7/GPIO36/FSPICLK/SUBSPICLK)
- net LORA_M1: now also J14.2 (Pin_2)
- net LORA_AUX: now reaches U2.31 (GPIO38/FSPIWP/SUBSPIWP)
- net LORA_AUX: now also J14.5 (Pin_5)
- net LORA_UART_TX: now reaches U2.36 (U0RXD/GPIO44/CLK_OUT2)
- net LORA_UART_TX: now also J14.4 (Pin_4)
- net LORA_UART_RX: now reaches U2.37 (U0TXD/GPIO43/CLK_OUT1)
- net LORA_UART_RX: now also J14.3 (Pin_3)
- no-connect marks 18 -> 13
Other:
- note added: "LORA"
- moved on the sheet: R19
